File: chip-breakout.kicad_pcb (KiCad board)
At the start: 2 copper layers, 94 x 76.2 mm, 15 parts

Commit message: including jlcpcb gerbers
Other:
- board text added: "https://github.com/cbluoss/package_breakout"
Changed lines of the file:
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@@
   (general
     (thickness 1.6)
-    (drawings 4)
+    (drawings 5)
     (tracks 732)
     (zones 0)
@@
       (layerselection 0x010fc_ffffffff)
       (usegerberextensions false)
-      (usegerberattributes false)
+      (usegerberattributes true)
       (usegerberadvancedattributes false)
       (creategerberjobfile false)
@@
       (plotinvisibletext false)
       (padsonsilk false)
-      (subtractmaskfromsilk false)
+      (subtractmaskfromsilk true)
       (outputformat 1)
       (mirror false)
-      (drillshape 1)
+      (drillshape 0)
       (scaleselection 1)
-      (outputdirectory ""))
+      (outputdirectory "gerbers"))
   )
   (net 0 "")
@@
     )
   )
+  (gr_text https://github.com/cbluoss/package_breakout (at 119.38 84.455) (layer B.SilkS)
+    (effects (font (size 1 1) (thickness 0.15)) (justify mirror))
+  )
   (gr_line (start 49.53 26.67) (end 49.53 102.87) (layer Edge.Cuts) (width 0.05))
